File: telemetry-shorter.brd (EAGLE design)
At the start: 69.8 x 22.9 mm, 60 parts, among them SW1 B3U-1000P-2P-SMD, U1 ATSAMD21G18_QFN, U2 SPX3819M5-L-3-0, U3 MCP73831T-2ACI/OT, U4 MPU-9250, U5 SIM868, U6 BMP280, X1 JSTPH, X2 32.768, X3 ZX62-B-5PA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

Commit message: Small fixes
Parts:
- moved JP2 0.06 mm to (57.2, 3.24)
- moved TP13 0.06 mm to (61.3, 3.11)
- moved TP6 0.06 mm to (59.2, 3.11)
Other:
- outline, holes or cut-outs redrawn

Commit message: Updated for MacroFab
Parts:
- removed L1: RED-0805, Seeed-LED-2016:LED-0805
- removed L3: CLEAR-BLUE-0805, Seeed-LED-2016:LED-0805
- added D3: MF-LED-0603-GREEN, MF_LEDs:LED0603
- added D4: MF-LED-0603-RED, MF_LEDs:LED0603
- D1: value MBR120 -> MBR120ESFT3G
- SW1: value B3U-1000P-2P-SMD -> MF-SW-TACT-4.2MM; device Seeed-Switch-2016:SW2-2.6-3.0X2.5X1.2+0.4MM -> MF_Switches:TACT4.2MM
- U1: value ATSAMD21G18_QFN -> ATSAMD21G18A-MUT
- X1: value JSTPH -> S2B-PH-SM4-TB(LF)(SN)
- X2: value 32.768 -> FC-135 32.7680KA-A3
- X3: value ZX62-B-5PA -> MF-CON-MICROUSB-RIGHT; device Deegou-Connectors:MICRO-USB5+6P-SMD-0.65-AB -> MF_Connectors:MICROUSB-RIGHT
- X5, X6: value U-FL -> U.FL-R-SMT(10)
- moved SW1 0.46 mm to (8.26, 7.18)
- moved X3 0.38 mm to (2.67, 11.4)
Connections:
- new net SLD: X3.S1, X3.S2, X3.S3, X3.S4, X3.S5, X3.S6
- net !RESET: now also SW1.P$1, SW1.P$2; no longer SW1.1
- net GND: now also D4.CATHODE, SW1.P$3, SW1.P$4; no longer L1.-, SW1.2, X3.P1, X3.P2, X3.P3, X3.P4, X3.P5, X3.P6
- net N$1: now also D3.CATHODE; no longer L3.-
- net N$8: now also D4.ANODE; no longer L1.+
- net VBUS: now also D3.ANODE; no longer L3.+
Routing:
- net GND: track 171.0 -> 146.0 mm, vias 73 -> 80
- net !RESET: track 23.6 -> 25.9 mm
- net SIM_VDD: track 11.8 -> 10.3 mm
- net D-: track 22.3 -> 23.5 mm
- net N$1: track 2.33 -> 3.10 mm
- net N$8: track 5.44 -> 6.01 mm
- net VBUS: track 43.3 -> 43.8 mm, vias 5 -> 3
- net D+: track 25.5 -> 26.0 mm
Other:
- outline, holes or cut-outs redrawn
