File: telemetry-shorter.brd (EAGLE design)
At the start: 69.8 x 22.9 mm, 62 parts, among them SW1 MF-SW-TACT-4.2MM, U1 ATSAMD21G18A-MUT, U2 SPX3819M5-L-3-0, U3 MCP73831T-2ACI/OT, U4 MPU-9250, U5 SIM868, U6 BMP280, X1 S2B-PH-SM4-TB(LF)(SN), X2 FC-135 32.7680KA-A3, X3 MF-CON-MICROUSB-RIGHT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

Commit message: Added logo to back
Parts:
- moved TP7 0.63 mm to (63.9, 10.0)
Routing:
- net VDD_EXT_2V8: track 18.3 -> 19.0 mm
Other:
- board text added: "FAR"
- board text added: "FROM"
- board text added: "Forschungsgemeinschaft Alternative Raumfahrt"
- board text added: "HOME"
